File: stm32f072_template.kicad_sch (KiCad schematic)
At the start: 23 parts, among them J1 USB_C_Receptacle_USB2.0, J2 Conn_01x20, J3 Conn_01x20, U1 STM32F072CBT6, U2 PRTR5V0U2X

Commit message: replace USB footprint
Parts:
- J1: footprint Connector_USB:USB_C_Receptacle_HRO_TYPE-C-31-M-12 -> PCM_marbastlib-various:USB_C_Receptacle_HRO_TYPE-C-31-M-12
